File: BikeLoad/BikeLoad.kicad_sch (KiCad schematic)
At the start: 0 parts

Commit message: .
Parts:
- added A1: Arduino_UNO_R3, Module:Arduino_UNO_R3, symbol MCU_Module:Arduino_UNO_R3
- added C1, C2: C, symbol Device:C
- added C3, C4: C_Polarized, symbol Device:C_Polarized
- added D1: BZV55B51, Diode_SMD:D_MiniMELF, symbol Diode:BZV55B51
- added J1: DC Input, symbol Connector_Generic:Conn_01x02
- added J2: Hall Input, symbol Connector:Conn_01x06_Pin
- added J3: Pot Input, symbol Connector:Conn_01x03_Pin
- added J4: DC Out, symbol Connector_Generic:Conn_01x02
- added J5: Control, symbol Connector:Conn_01x02_Pin
- added Q2: PNP, symbol Simulation_SPICE:PNP
- added R1, R10, R11, R5, R6, R7, R8, R9: R, symbol Device:R
- added R13, R2, R3, R4: 10k, symbol Device:R
- added U1: ACS770xCB-050U-PFF, Sensor_Current:Allegro_CB_PFF, symbol Sensor_Current:ACS770xCB-050U-PFF
- added U2: TPSM5601R5HRDAR, TPSM5601R5HRDAR:IC_TPSM5601R5HRDAR, symbol TPSM5601R5HRDAR:TPSM5601R5HRDAR
- added U3: L7805, symbol Regulator_Linear:L7805
Connections:
- new net: Q2.1 (C), R11.1
- new net: J3.2 (Pin_2), R1.1
- new net: D1.1 (K), Q2.2 (B), R13.1
- new net: R8.2, R9.1
- new net: R5.2, R6.1, U2.9 (FB)
- new net: R7.2, R8.1
- new net: J1.1 (Pin_1), R7.1, U1.4 (IP+)
- new net +5V: C4.1, J2.1 (Pin_1), R2.1, R3.1, R4.1, R5.1, U1.1 (VCC), U2.7 (VOUT), U2.8 (VOUT__1)
- new net DC_metered: C2.1, C3.1, J4.1 (Pin_1), Q2.3 (E), R13.2, U1.5 (IP-), U2.1 (VIN), U2.14 (VIN__1), U2.2 (EN)
- new net GND: C1.2, C2.2, C3.2, C4.2, D1.2 (A), J1.2 (Pin_2), J2.2 (Pin_2), J3.3 (Pin_3), J4.2 (Pin_2), R10.2, R11.2, R6.2, U1.2 (GND), U2.10 (AGND), U2.15 (PGND)
- new net Hall_A: J2.3 (Pin_3), R2.2
- new net Hall_B: J2.4 (Pin_4), R3.2
- new net Hall_C: J2.5 (Pin_5), R4.2
- new net InputCurrent: U1.3 (VIOUT)
- new net InputPot: C1.1, R1.2
- new net InputVoltage: R10.1, R9.2
- no-connect marks 0 -> 7
Other:
- note added: "Output to load transistor"

Commit message: schematic
Parts:
- removed J5: Control, symbol Connector:Conn_01x02_Pin
- removed R7, R8: R, symbol Device:R
- removed U3: L7805, symbol Regulator_Linear:L7805
- added C5, C6: 1, symbol Device:C_Polarized
- added C8: 10u, symbol Device:C_Polarized
- added D2, D3, D4: BZV55B4V3, Diode_SMD:D_MiniMELF, symbol Diode:BZV55B4V3
- added D5, D6: D, symbol Device:D
- added J6: DC out, symbol Connector_Generic:Conn_01x02
- added J7: LoadControl, symbol Connector_Generic:Conn_01x02
- added Q1: PNP, symbol Simulation_SPICE:PNP
- added R12, R15, R16, R17, R18: R, symbol Device:R
- added R14: 10k, symbol Device:R
- added U4: R-785.0-1.0, Converter_DCDC:Converter_DCDC_RECOM_R-78E-0.5_THT, symbol Regulator_Switching:R-785.0-1.0
- C4: value C_Polarized -> 1
- J4: value DC Out -> Load
Connections:
- net +5V: now also A1.5 (+5V), Q1.1 (C), R16.1, U4.3 (OUT); no longer C4.1, R5.1, U2.7 (VOUT), U2.8 (VOUT__1)
- net GND: now also A1.29 (GND), A1.6 (GND), A1.7 (GND), C6.2, C8.2, D4.2 (A), J6.2 (Pin_2), J7.2 (Pin_2), R18.2, U4.2 (GND); no longer C4.2
- net Hall_A: now also A1.19 (D4)
- net Hall_B: now also A1.20 (D5)
- net Hall_C: now also A1.21 (D6)
- net InputCurrent: now also A1.10 (A1)
- net InputPot: now also A1.12 (A3)
- net InputVoltage: now also A1.9 (A0)
- net TempSensor: now reaches A1.11 (A2)
- net SCapVolts: now reaches A1.13 (SDA/A4)
- net SCapVolts: now also R17.2, R18.1
- net PWMout: now reaches A1.24 (D9)
- net PWMout: now also R15.1, R16.2
- net LEDenable: now reaches A1.25 (D10)
- net LEDserial: now reaches A1.26 (D11)
- net at R9.1: now also J1.1 (Pin_1), U1.4 (IP+)
- new net: C8.1, J7.1 (Pin_1), R14.2
- new net: C4.1, D2.1 (K), D6.2 (A), R12.2, R17.1
- new net: C4.2, C5.1, D2.2 (A), D3.1 (K)
- new net: D5.1 (K), D6.1 (K), U4.1 (IN)
- new net: Q1.2 (B), R15.2
- new net: Q1.3 (E), R14.1
- new net: C5.2, C6.1, D3.2 (A), D4.1 (K)
- new net +13V: D5.2 (A), J6.1 (Pin_1), R12.1, R5.1, U2.7 (VOUT), U2.8 (VOUT__1)
- no-connect marks 7 -> 22
Other:
- note added: "For 12 VDC car chager"
- moved on the sheet: A1, C1, C2, C3, C4, D1, J2, J3, Q2, R1, R10, R11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

Commit message: .
Parts:
- added C7: C, Capacitor_SMD:C_0805_2012Metric, symbol Device:C
- added H1, H2, H3, H4: MountingHole, MountingHole:MountingHole_3.2mm_M3, symbol Mechanical:MountingHole
- added J5: Temp sensor, Connector_PinHeader_2.54mm:PinHeader_1x02_P2.54mm_Vertical, symbol Connector:Conn_01x02_Pin
- added R7: 10k, Resistor_SMD:R_0805_2012Metric, symbol Device:R
- added R8: 1k, Resistor_SMD:R_0805_2012Metric, symbol Device:R
- added TP1, TP2, TP4: TestPoint, TestPoint:TestPoint_Loop_D1.80mm_Drill1.0mm_Beaded, symbol Connector:TestPoint
- added TP3: TestPoint, TestPoint:TestPoint_2Pads_Pitch2.54mm_Drill0.8mm, symbol Connector:TestPoint
- C1, C2: footprint (none) -> Capacitor_SMD:C_0805_2012Metric
- C3, C8: footprint (none) -> Capacitor_THT:CP_Radial_D5.0mm_P2.00mm
- C4, C5, C6: footprint (none) -> Capacitor_THT:CP_Radial_D8.0mm_P5.00mm
- D5, D6: footprint (none) -> Diode_SMD:D_SOD-123
- J1, J4, J6: footprint (none) -> Connector_Phoenix_MSTB:PhoenixContact_MSTBVA_2,5_2-G-5,08_1x02_P5.08mm_Vertical
- J2: footprint (none) -> Connector_PinHeader_2.54mm:PinHeader_1x06_P2.54mm_Vertical
- J3: footprint (none) -> Connector_PinHeader_2.54mm:PinHeader_1x03_P2.54mm_Vertical
- J7: footprint (none) -> Connector_PinHeader_2.54mm:PinHeader_1x02_P2.54mm_Vertical
- Q1: value PNP -> BC556; footprint (none) -> Package_TO_SOT_THT:TO-92
- Q2: footprint (none) -> Package_TO_SOT_THT:TO-220-3_Vertical
- R1, R13, R15, R16, R17, R18, R2, R3, R4, R5, R6: footprint (none) -> Resistor_SMD:R_0805_2012Metric
- R10, R9: footprint (none) -> Resistor_SMD:R_0815_2038Metric
- R11: footprint (none) -> Resistor_THT:R_Axial_DIN0207_L6.3mm_D2.5mm_P15.24mm_Horizontal
- R12, R14: footprint (none) -> Resistor_THT:R_Axial_DIN0207_L6.3mm_D2.5mm_P10.16mm_Horizontal
Connections:
- net +13V: now also TP1.1
- net +5V: now also Q1.3 (E), R7.1, TP2.1; no longer Q1.1 (C)
- net GND: now also C7.2, J5.2 (Pin_2), TP3.1
- net TempSensor: now also C7.1, R8.2
- net at C4.1, D2.1 (K), D6.2 (A)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: now also TP4.1
- net at R11.1: now also Q2.2 (C); no longer Q2.1 (C)
- net at D1.1 (K), R13.1: now also Q2.1 (B); no longer Q2.2 (B)
- net at R14.1: now also Q1.1 (C); no longer Q1.3 (E)
- new net: J5.1 (Pin_1), R7.2, R8.1
Other:
- moved on the sheet: C1, J2, J3, R1, R2, R3, R4
